Commit message: 27.12.2025

File: resources/PAROL6.urdf (robot description, URDF)
Before this commit: robot parol6, 8 links, 7 joints
Links:
- added link tcp_link, mass 0.001; visual sphere radius=0.005
Joints:
- added joint joint_tcp: type fixed, parent L6, child tcp_link, origin xyz=0 0 0.15 rpy=0 1.5708 0

Commit message: 2.01.2026

File: resources/PAROL6.urdf (robot description, URDF)
Before this commit: robot parol6, 9 links, 8 joints
Links:
- removed link tcp_link
Joints:
- removed joint joint_tcp
